Commit message: refactor: update vehicle wheelbase and camera pitch angle parameters to match real hardware specifications

File: vehicles/sample_vehicle/xacro/ai_car1.xacro (robot description, xacro)
@@ -9,4 +9,6 @@
   <xacro:property name="WHEEL_RADIUS" value="0.12"/>
   <xacro:property name="CASTER_RADIUS" value="0.10"/>
+  <!-- Front drive-wheel axle to rear caster axle. -->
+  <xacro:property name="WHEELBASE" value="0.815"/>
   <xacro:property name="BASE_FOOTPRINT" value="base_footprint"/>
   <xacro:property name="BASE" value="base"/>
@@ -45,5 +47,5 @@
   <xacro:caster_back_joint_macro
     caster_back="${CASTER_BACK}" parent="${BASE}"
-    x="-0.76" y="0.0" z="${CASTER_RADIUS}"
+    x="-${WHEELBASE}" y="0.0" z="${CASTER_RADIUS}"
     roll="${90.0*D2R}" pitch="0.0" yaw="${90.0*D2R}"/>
   <xacro:caster_back_link_macro
