Commit message: feat: six-lane only driving, speed limit knob, remove QP/UFLD/odom_imu_localizer
- Remove the lap-map + QP raceline method (lane_navigator, QP modules, launches,
  sim LaneNavigator/map panel), UFLD (backend, ufld/, exporter, sim button),
  odom_imu_localizer and the aggregate launches (all_system_2027, all_robot_nodes,
  3_bringup_all_nodes.sh). Only hardware + six_lane launches remain
  (bash/1_bringup_hardware.sh, bash/2_six_lane.sh, make six-lane).
- Single manual knob speed_limit (0.3-3.0 m/s) for real vehicle (launch arg,
  topic, param) and simulator (HUD slider, also published to ROS); lookahead,
  lost_timeout and cone-avoid distances auto-scale with it (effective_control).
- Add detection-latency compensation, distance-based command hold and a
  wheel+IMU speed estimator; JS mirror in web_simulator with golden-data parity
  test (web_simulator/test/parity.html).
- Unify wheel diameter to 0.254 m (xacro WHEEL_RADIUS 0.127, BASE_HEIGHT 0.12).
- Rename lane_nav -> lane_core, twist_mux input mpc -> autonomous,
  cmd_vel topic -> /aiformula_control/six_lane_planner/cmd_vel.
- Split pure cores (motor_math) and add tests; drop stale topics/docs;
  rewrite CLAUDE.md requirements and add docs/README.md.

Co-Authored-By: Claude Sonnet 5.5 <noreply@anthropic.com>

File: vehicles/sample_vehicle/xacro/ai_car1.xacro (robot description, xacro)
@@ -7,5 +7,8 @@
   <xacro:property name="PI" value="3.1415926"/>
   <xacro:property name="D2R" value="${PI/180}"/>
-  <xacro:property name="WHEEL_RADIUS" value="0.12"/>
+  <!-- 車輪半径 = config/wheel.yaml の diameter 0.254 / 2 (motor_controller / odometry の速度換算と同じ) -->
+  <xacro:property name="WHEEL_RADIUS" value="0.127"/>
+  <!-- base_link の地上高 (実測. ZED X の高さ 0.12 + 0.44 = 0.56 m の基準. 車輪半径とは別) -->
+  <xacro:property name="BASE_HEIGHT" value="0.12"/>
   <xacro:property name="CASTER_RADIUS" value="0.10"/>
   <!-- Front drive-wheel axle to rear caster axle. -->
@@ -22,5 +25,5 @@
   <xacro:base_macro
     base="${BASE}" parent_link="${BASE_FOOTPRINT}"
-    x="0.0" y="0.0" z="${WHEEL_RADIUS}"
+    x="0.0" y="0.0" z="${BASE_HEIGHT}"
     roll="0.0" pitch="0.0" yaw="${180.0*D2R}"/>
   <!-- zedx -->
@@ -30,5 +33,5 @@
   <xacro:wheel_joint_macro
     wheel="${WHEEL_LEFT}" parent="${BASE}"
-    x="0.0" y="0.3" z="${WHEEL_RADIUS}"
+    x="0.0" y="0.3" z="${BASE_HEIGHT}"
     roll="${90.0*D2R}" pitch="0.0" yaw="${90.0*D2R}"/>
   <xacro:wheel_link_macro
@@ -38,5 +41,5 @@
   <xacro:wheel_joint_macro
     wheel="${WHEEL_RIGHT}" parent="${BASE}"
-    x="0.0" y="-0.3" z="${WHEEL_RADIUS}"
+    x="0.0" y="-0.3" z="${BASE_HEIGHT}"
     roll="${90.0*D2R}" pitch="0.0" yaw="${90.0*D2R}"/>
   <xacro:wheel_link_macro

File: vehicles/sample_vehicle/xacro/parts/wheel_macro.xacro (robot description, xacro)
@@ -16,5 +16,5 @@
     <xacro:property name="MESH_FILE" value="package://sample_vehicle/xacro/meshes/tire.dae"/>
     <xacro:property name="THICKNESS_SCALE" value="0.05"/>
-    <xacro:property name="SIZE_SCALE" value="0.12"/>
+    <xacro:property name="SIZE_SCALE" value="0.127"/>  <!-- 車輪半径 [m] = wheel.yaml diameter / 2 -->
     <link name="${wheel}_link">
       <visual>
